File: anglesenseor.brd (EAGLE design)
At the start: 50 x 12 mm, 29 parts, among them X1 MPT0.5/4-2.54, X2 MPT0.5/4-2.54

Commit message: routed
Parts:
- removed H3, H4: (no value), diskreetit:CHIPLED_0603
- added C8, C9: 100n, passiivit:C0603
- added R12, R13: 1k00, passiivit:R0603
- added X3: B4B-PH-K-S, liittimet:B4B-PH-K-S
- D1: value OMAT_IC_2_IIS328DQTR -> IIS328DQTR; device cpu:OMAT_IC_2_QFN50P400X400X100-25N -> piirit:QFN50P400X400X100-25N
- D3: value PCA9632 -> PCA9536DGK; device piirit:MSOP-10 -> piirit:TSSOP8-66
- R7, R8: value 1k00 -> 10k0
- X1, X2: value MPT0.5/4-2.54 -> S4B-PH-SM4-TB; device cpu:MPT0.5/4-2.54 -> liittimet:JST-PH2.0-RA-4
- moved U$1 74.5 mm to (44.8, 10.1)
- moved R9 17.8 mm to (15.0, 18.5), flipped to the bottom, turned to 180 degrees
- moved R8 17.3 mm to (23.5, 12.0), flipped to the bottom, turned to 90 degrees
- moved R11 16.8 mm to (18.0, 18.5), flipped to the bottom, turned to 180 degrees
- moved C7 13.1 mm to (27.5, 18.5), flipped to the bottom, turned to 180 degrees
- moved D3 13.1 mm to (27.5, 16.0), flipped to the bottom
- moved R4 11.5 mm to (11.5, 13.0), flipped to the bottom, turned to 180 degrees
- moved R7 11.4 mm to (28.0, 12.0), flipped to the bottom, turned to 90 degrees
- moved R10 11.2 mm to (12.0, 18.5), flipped to the bottom, turned to 180 degrees
- moved C6 10.8 mm to (18.0, 16.0), flipped to the bottom, turned to 270 degrees
- moved R1 10.6 mm to (20.0, 16.0), flipped to the bottom, turned to 90 degrees
- moved D2 9.19 mm to (15.5, 14.5), flipped to the bottom, turned to 270 degrees
- moved X2 8.73 mm to (49.5, 10.0), flipped to the bottom
- moved R2 8.14 mm to (21.5, 16.0), flipped to the bottom, turned to 90 degrees
- moved C2 7.83 mm to (21.0, 4.50), flipped to the bottom, turned to 270 degrees
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Connections:
- removed net N$10: H3.A, R6.1
- removed net N$11: H2.A, R7.1
- removed net N$12: H1.A, R8.1
- removed net N$13: D3.4, H1.C
- removed net N$14: D3.3, H2.C
- removed net N$15: D3.2, H3.C
- removed net N$16: D3.1, H4.C
- removed net N$2: D2.7, R3.1, X1.2, X2.3
- removed net N$3: D2.10, R4.1, X1.4, X2.1
- removed net N$5: D1.16, D2.8, D3.9, R2.1
- removed net N$6: D1.11, D2.9, D3.8, R1.1
- new net IN1: C9.1, D3.3, R12.1
- new net IN2: C8.1, D3.5, R13.1
- new net IN_1: R12.2, R7.1, X3.1
- new net IN_2: R13.2, R8.1, X3.3
- new net LED1: D3.1, H1.C
- new net LED2: D3.2, H2.C
- new net N$8: H2.A, R6.1
- new net SCL3V3: D1.11, D2.9, D3.6, R1.1
- new net SCL5V: D2.10, R4.1, X1.4, X2.4
- new net SDA3V3: D1.16, D2.8, D3.7, R2.1
- new net SDA5V: D2.7, R3.1, X1.2, X2.2
- net +3V3: now also D3.8; no longer D3.10
- net +5V: now also X2.1; no longer X2.4
- net GND: now also C8.2, C9.2, D3.4, X2.3, X3.2, X3.4; no longer D3.5, D3.6, D3.7, X2.2
- net N$9: now also H1.A; no longer H4.A
Routing:
- net +5V: track 0.00 -> 78.1 mm, vias 0 -> 5
- net +3V3: track 0.00 -> 66.1 mm, vias 0 -> 3
- net SCL5V: track 0.00 -> 60.2 mm, vias 0 -> 2
- net SDA5V: track 0.00 -> 51.4 mm, vias 0 -> 2
- net SDA3V3: track 0.00 -> 37.1 mm
- net SCL3V3: track 0.00 -> 25.9 mm, vias 0 -> 2
- net GND: track 0.00 -> 13.5 mm, vias 0 -> 20
- net LED1: track 0.00 -> 13.2 mm, vias 0 -> 1
- net LED2: track 0.00 -> 7.66 mm, vias 0 -> 1
- net IN1: track 0.00 -> 5.40 mm
- net N$7: track 0.00 -> 3.93 mm
- net IN2: track 0.00 -> 3.86 mm
- net IN_2: track 0.00 -> 3.53 mm
- net N$4: track 0.00 -> 3.49 mm
- net IN_1: track 0.00 -> 3.33 mm
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- added copper zone on layer 1, net GND
- added copper zone on layer 16, net GND
Other:
- board size 50 x 12 mm -> 50 x 19.8 mm
- board text added: "(C) KIMMOLI 2018"
- board text added: "+5V"
- board text added: "ANGLE SENSOR LIMIT SWITCH IO"
- board text added: "GND"
- board text added: "IN1"
- board text added: "IN2"
- board text added: "SCL"
- board text added: "SDA"
- board text added: "TELAKONE"

Commit message: mutteri
Parts:
- moved H1 3.26 mm to (31.3, 8.60), turned to 0 degrees
- moved H2 3.26 mm to (31.3, 11.4), turned to 0 degrees
- moved R5 2.80 mm to (35.5, 6.28), flipped to the bottom, turned to 180 degrees
- moved R6 2.20 mm to (36.1, 13.7), flipped to the bottom, turned to 180 degrees
Routing:
- net +5V: track 78.1 -> 87.8 mm
- net N$8: track 1.52 -> 5.75 mm, vias 0 -> 1
- net SDA5V: track 51.4 -> 55.2 mm
- net N$9: track 1.74 -> 4.76 mm, vias 0 -> 1
- net LED1: track 13.2 -> 11.1 mm
- net +3V3: track 66.1 -> 64.5 mm
- net SCL5V: track 60.2 -> 61.3 mm
- net LED2: track 7.66 -> 6.87 mm
- net GND: vias 20 -> 15
Other:
- board text added: "1 +5V 2 SDA 3 GND 4 SCL"
- board text removed: "+5V"
- board text removed: "SCL"
- board text removed: "SDA"

Commit message: more gnd, finalise
Parts:
- moved H1 0.20 mm to (31.3, 8.40)
- moved C7 0.10 mm to (27.5, 18.4)
- moved R10 0.10 mm to (12.0, 18.4)
- moved R11 0.10 mm to (18.0, 18.4)
- moved R9 0.10 mm to (15.0, 18.4)
- moved U$1 0.10 mm to (44.8, 9.95)
- moved C5 0.10 mm to (11.3, 4.80)
- moved R5 0.10 mm to (35.5, 6.18)
- moved C3 0.10 mm to (15.0, 1.90)
- moved C1 0.10 mm to (29.0, 4.40)
- moved C2 0.10 mm to (21.0, 4.40)
- moved C4 0.10 mm to (15.0, 7.40)
- moved C6 0.10 mm to (18.0, 15.9)
- moved C8 0.10 mm to (26.5, 11.9)
- moved C9 0.10 mm to (31.0, 11.9)
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Routing:
- net GND: track 13.5 -> 17.1 mm, vias 15 -> 34
