File: anglesenseor.sch (EAGLE design)
At the start: 29 parts, among them X1 MPT0.5/4-2.54, X2 MPT0.5/4-2.54

Commit message: routed
Parts:
- removed H3, H4: (no value), diskreetit:LEDCHIPLED_0603
- added C8, C9: 100n, passiivit:CAP0603
- added R12, R13: 1k00, passiivit:RES0603
- added X3: B4B-PH-K-S, liittimet:B4B-PH-K-S
- D1: value OMAT_IC_2_IIS328DQTR -> IIS328DQTR; device cpu:OMAT_IC_2_IIS328DQTR -> piirit:IIS328DQTR
- D3: value PCA9632 -> PCA9536DGK; device piirit:PCA9632 -> piirit:PCA9536DGK
- R7, R8: value 1k00 -> 10k0
- X1, X2: value MPT0.5/4-2.54 -> S4B-PH-SM4-TB; device cpu:MPT0.5/4-2.54 -> liittimet:S4B-PH-SM4-TB
Connections:
- net N$5 renamed SDA3V3
- net N$6 renamed SCL3V3
- removed net N$10: H3.A, R6.1
- removed net N$11: H2.A, R7.1
- removed net N$12: H1.A, R8.1
- removed net N$13: D3.LED3, H1.C
- removed net N$14: D3.LED2, H2.C
- removed net N$15: D3.LED1, H3.C
- removed net N$16: D3.LED0, H4.C
- removed net N$2: D2.SDAIN, R3.1, X1.2, X2.3
- removed net N$3: D2.SCLIN, R4.1, X1.4, X2.1
- new net IN1: C9.1, D3.IO2, R12.1
- new net IN2: C8.1, D3.IO3, R13.1
- new net IN_1: R12.2, R7.1, X3.1
- new net IN_2: R13.2, R8.1, X3.3
- new net LED1: D3.IO0, H1.C
- new net LED2: D3.IO1, H2.C
- new net N$8: H2.A, R6.1
- new net SCL5V: D2.SCLIN, R4.1, X1.4, X2.4
- new net SDA5V: D2.SDAIN, R3.1, X1.2, X2.2
- net +5V: now also X2.1; no longer X2.4
- net GND: now also C8.2, C9.2, X2.3, X3.2, X3.4; no longer D3.A0, D3.A1, X2.2
- net N$9: now also H1.A; no longer H4.A
Other:
- moved on the sheet: C7, H1, H2, R5, R6, R7, R8, X2
